Commit message: changed node for real robot

File: src/piper_description/urdf/piper_description.urdf (robot description, URDF)
Before this commit: robot piper, 10 links, 9 joints
Joints:
- joint joint6_to_gripper_base: origin xyz=0 0 0 rpy=0 0 0 -> xyz=0 0 0 rpy=0 0 1.5708

File: src/piper_description/urdf/piper_description.xacro (robot description, xacro)
@@ -382,5 +382,5 @@
     <origin
       xyz="0 0 0"
-      rpy="0 0 0" />
+      rpy="0 0 1.5708" />
     <parent
       link="link6" />

Commit message: squelched joint state prints and updated joint limits in urdf

File: src/piper_description/urdf/piper_description.urdf (robot description, URDF)
Before this commit: robot piper, 10 links, 9 joints
Joints:
- joint joint6: limit lower=-2.0944 upper=2.0944 effort=100 velocity=3 -> lower=-0.5 upper=2.0 effort=100 velocity=3
